File: Hw/flat-sat/FlatSat.kicad_pcb (KiCad board)
At the start: 4 copper layers, 81 x 20 mm, 100 parts, among them J1 Antenna, J3 Conn_01x06_Female, P1 USB_C_Plug_USB2.0, SW1 SW, U1 AP2112K-3.3, U2 RFSW8006QTR7, U3 RP2040, U4 0900PC15A0036, U5 0900FM15D0039, U6 PE42421, U7 SX1262IMLTRT, U8 CC1352P1F3RGZT, U9 W25Q16JV, Y1 48MHz, Y2 32.768kHz, Y3 32Mhz, Y4 12MHz

Commit message: Remove previous layout, update gitignore
Parts:
- removed BOOT1, RESET1, RESET_CC1, SW1: SW, CatSniffer:TS1088R02026
- removed C1, C37: 1uF, Capacitor_SMD:C_0603_1608Metric
- removed C10, C11, C12, C13, C15, C16, C32: 100nF, Capacitor_SMD:C_0402_1005Metric
- removed C14, C17: 22uF, Capacitor_SMD:C_0603_1608Metric
- removed C18, C19: 22pF, Capacitor_SMD:C_0603_1608Metric
- removed C2, C21, C24, C29: 0.1uF, Capacitor_SMD:C_0603_1608Metric
- removed C20, C23, C27, C6, C7, C8, C9: 100pF, Capacitor_SMD:C_0603_1608Metric
- removed C22: 47pF, Capacitor_SMD:C_0603_1608Metric
- removed C25, C26: 3.3pF, Capacitor_SMD:C_0603_1608Metric
- removed C28, C4: 27pF, Capacitor_SMD:C_0402_1005Metric
- removed C3, C38: 1uF, Capacitor_SMD:C_0402_1005Metric
- removed C30, C39, C40, C41, C42, C43, C44, C45, C46, C5: 0.1uF, Capacitor_SMD:C_0402_1005Metric
- removed C31, C35: 1nF, Capacitor_SMD:C_0603_1608Metric
- removed C33: 470nF, Capacitor_SMD:C_0603_1608Metric
- removed C34, C36: 10pF, Capacitor_SMD:C_0603_1608Metric
- removed D1, D2, D3, D4: LED, LED_SMD:LED_0603_1608Metric_Pad1.05x0.95mm_HandSolder
- removed F1: 0.5A, Fuse:Fuse_0805_2012Metric_Pad1.15x1.40mm_HandSolder
- removed G***: LOGO, Aesthetics:electronic_cats_logo_4x3
- removed G***: LOGO, CatSniffer:calderon
- removed G***: LOGO, Aesthetics:electronic_cats_logo_8x6
- removed G***: LOGO, CatSniffer:calderon_7.5x7.5
- removed J1: Antenna, bast-wan:SMA_EDGE
- removed J3: Conn_01x06_Female, Connector:Tag-Connect_TC2030-IDC-NL_2x03_P1.27mm_Vertical
- removed JP1: Jumper, Jumper:SolderJumper-3_P1.3mm_Bridged12_RoundedPad1.0x1.5mm_NumberLabels
- removed L1: BLM18HE152SN1D, Inductor_SMD:L_0603_1608Metric
- removed L2: 6.8uH, Inductor_SMD:L_0603_1608Metric
- removed L3: 9.1nH, Inductor_SMD:L_0603_1608Metric
- removed L4: 47nH, Inductor_SMD:L_0603_1608Metric
- removed L5: 15uH, Inductor_SMD:L_0603_1608Metric
- removed P1: USB_C_Plug_USB2.0, Connectors:C393939
- removed R1, R2: 5k1, Resistor_SMD:R_0603_1608Metric
- removed R10, R11: 27, Resistor_SMD:R_0402_1005Metric
- removed R12: 1k, Resistor_SMD:R_0402_1005Metric
- removed R13: 10k, Resistor_SMD:R_0402_1005Metric
- removed R3, R4, R5, R9: 330, Resistor_SMD:R_0603_1608Metric
- removed R6: 100K, Resistor_SMD:R_0603_1608Metric
- removed R7, R8: 100R, Resistor_SMD:R_0603_1608Metric
- removed REF** (x4): HOLE, CatSniffer:HOLE
- removed REF**: OSHW-Logo_5.7x6mm_SilkScreen, Symbol:OSHW-Logo_5.7x6mm_SilkScreen
- removed REF**: OSHW-Logo_7.5x8mm_SilkScreen, Symbol:OSHW-Logo_7.5x8mm_SilkScreen
- removed U1: AP2112K-3.3, Package_TO_SOT_SMD:SOT-23-5
- removed U2: RFSW8006QTR7, CatSniffer:SON50P200X200X90-9N
- removed U3: RP2040, Package_DFN_QFN:QFN-56-1EP_7x7mm_P0.4mm_EP3.2x3.2mm
- removed U4: 0900PC15A0036, CatSniffer:0900FM15D0039E
- removed U5: 0900FM15D0039, CatSniffer:0900FM15D0039E
- removed U6: PE42421, Package_TO_SOT_SMD:SOT-363_SC-70-6
- removed U7: SX1262IMLTRT, Package_DFN_QFN:QFN-24-1EP_4x4mm_P0.5mm_EP2.65x2.65mm
- removed U8: CC1352P1F3RGZT, Package_DFN_QFN:VQFN-48-1EP_7x7mm_P0.5mm_EP5.15x5.15mm_ThermalVias
- removed U9: W25Q16JV, CatSniffer:W25Q16JVUUIQ
- removed Y1: 48MHz, Crystal:Crystal_SMD_3225-4Pin_3.2x2.5mm
- removed Y2: 32.768kHz, Crystal:Crystal_SMD_2012-2Pin_2.0x1.2mm
- removed Y3: 32Mhz, Crystal:Crystal_SMD_2520-4Pin_2.5x2.0mm
- removed Y4: 12MHz, Crystal:Crystal_SMD_3225-4Pin_3.2x2.5mm
Routing:
- net GND: track 425.9 -> 0.00 mm, vias 101 -> 0
- net +3V3: track 101.1 -> 0.00 mm, vias 16 -> 0
- net /BOOT: track 98.9 -> 0.00 mm, vias 3 -> 0
- net /RESET_CC: track 67.8 -> 0.00 mm, vias 3 -> 0
- net /CTF2: track 59.1 -> 0.00 mm, vias 4 -> 0
- net /CTF1: track 58.6 -> 0.00 mm, vias 2 -> 0
- net /VDDS: track 57.4 -> 0.00 mm, vias 6 -> 0
- net /CTF3: track 50.8 -> 0.00 mm, vias 2 -> 0
- net /cJTAG_TMSC: track 47.1 -> 0.00 mm, vias 1 -> 0
- net /cJTAG_TCK: track 44.4 -> 0.00 mm, vias 2 -> 0
- net /LED4: track 43.2 -> 0.00 mm, vias 2 -> 0
- net /TXD: track 42.7 -> 0.00 mm, vias 2 -> 0
- net /RXD: track 41.3 -> 0.00 mm, vias 2 -> 0
- net /DIO2: track 40.6 -> 0.00 mm, vias 2 -> 0
- net /ANT_SW: track 30.5 -> 0.00 mm, vias 2 -> 0
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- removed copper zone on F.Cu, net +3V3
- removed copper zone on In2.Cu, net +3V3
- removed copper zone on In2.Cu, net /VDDR
- removed copper zone on In2.Cu, net /VDDS
- removed copper zone on B.Cu, net GND
- removed copper zone on F.Cu, net GND
- removed copper zone on In1.Cu, net GND
Other:
- board outline removed
- board text removed: "&"
- board text removed: "CatSniffer V3.2"
- board text removed: "CatSniffer v3.2"
- board text removed: "electroniccats.com"
- board text removed: "pwnlab.com.mx"
